File: schematics/Z80Mini/Z80MiniFrame-Sound_Graphics/graphicsProcessor.sch (KiCad schematic (older format))
At the start: 27 parts, among them J2 COMP_VIDEOUT, J5 COMP_VIDEOIN, Q1 2N3904, U1 TMS9918A, U12 74LS32, U2 74LS574, U3 74LS574, U4 74LS574, U5 AS6C62256-55PCN, U6 74HC04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

Commit message: Testing C routines for VDP and keyboard. Generated backplane gerber files
Connections:
- net D0: now also U1.17 (CD7); no longer U1.24 (CD0)
- net D1: now also U1.18 (CD6); no longer U1.23 (CD1)
- net D2: now also U1.19 (CD5); no longer U1.22 (CD2)
- net D3: now also U1.20 (CD4); no longer U1.21 (CD3)
- net D4: now also U1.21 (CD3); no longer U1.20 (CD4)
- net D5: now also U1.22 (CD2); no longer U1.19 (CD5)
- net D6: now also U1.23 (CD1); no longer U1.18 (CD6)
- net D7: now also U1.24 (CD0); no longer U1.17 (CD7)
- net CPUCLK: now reaches U1.38 (CPUCLK)
- net A1 renamed A0
- no-connect marks 4 -> 3
Changed lines of the file:
@@
 Wire Wire Line
 	3950 4200 4050 4200
-NoConn ~ 3950 4100
 $Comp
 L Video:TMS9918A U1
@@
 	1250 3850 1350 3850
 Text HLabel 1100 5250 0    50   Input ~ 0
-A1
+A0
 Wire Wire Line
 	2550 5250 1100 5250
@@
 	3000 3500 1300 3500
 Text Label 2900 3050 0    50   ~ 0
+D0
+Text Label 2900 2950 0    50   ~ 0
+D1
+Text Label 2900 2850 0    50   ~ 0
+D2
+Text Label 2900 2750 0    50   ~ 0
+D3
+Text Label 2900 2650 0    50   ~ 0
+D4
+Text Label 2900 2550 0    50   ~ 0
+D5
+Text Label 2900 2450 0    50   ~ 0
+D6
+Text Label 2900 2350 0    50   ~ 0
 D7
-Text Label 2900 2950 0    50   ~ 0
-D6
-Text Label 2900 2850 0    50   ~ 0
-D5
-Text Label 2900 2750 0    50   ~ 0
-D4
-Text Label 2900 2650 0    50   ~ 0
-D3
-Text Label 2900 2550 0    50   ~ 0
-D2
-Text Label 2900 2450 0    50   ~ 0
-D1
-Text Label 2900 2350 0    50   ~ 0
-D0
 Text Label 6000 5650 0    50   ~ 0
 AD7
@@
 Text Label 7850 2350 0    50   ~ 0
 VD0
-Wire Bus Line
-	7700 3000 9250 3000
 Wire Wire Line
 	7800 2550 8000 2550
@@
 Entry Wire Line
 	7700 2650 7800 2550
-Connection ~ 7700 3000
 Text Label 7100 3800 0    50   ~ 0
 VA13
@@
 	1    0    0    -1
 $EndComp
+$Comp
+L 74xx:74LS574 U3
+U 1 1 5D7A0CA0
+P 6600 3600
+F 0 "U3" H 6600 4581 50  0000 C CNN
+F 1 "74LS574" H 6600 4490 50  0000 C CNN
+F 2 "Package_DIP:DIP-20_W7.62mm_Socket_LongPads" H 6600 3600 50  0001 C CNN
+F 3 "http://www.ti.com/lit/gpn/sn74LS574" H 6600 3600 50  0001 C CNN
+	1    6600 3600
+	1    0    0    -1
+$EndComp
+$Comp
+L Device:CTRIM CV1
+U 1 1 5DF8BFF1
+P 1350 2850
+F 0 "CV1" V 1603 2850 50  0000 C CNN
+F 1 "5-50pF" V 1512 2850 50  0000 C CNN
+F 2 "Potentiometer_THT:Potentiometer_ACP_CA9-V10_Vertical" H 1350 2850 50  0001 C CNN
+F 3 "~" H 1350 2850 50  0001 C CNN
+	1    1350 2850
+	0    -1   -1   0
+$EndComp
+Connection ~ 1750 2850
+$Comp
+L power:GND #PWR0129
+U 1 1 5E069747
+P 1750 3150
+F 0 "#PWR0129" H 1750 2900 50  0001 C CNN
+F 1 "GND" H 1755 2977 50  0000 C CNN
+F 2 "" H 1750 3150 50  0001 C CNN
+F 3 "" H 1750 3150 50  0001 C CNN
+	1    1750 3150
+	1    0    0    -1
+$EndComp
+Wire Wire Line
+	2450 2550 2450 3200
+Wire Wire Line
+	2450 3200 3000 3200
+Wire Wire Line
+	3000 3300 1950 3300
+Wire Wire Line
+	1950 3300 1950 2850
+Wire Wire Line
+	1950 2850 1750 2850
+Text HLabel 3150 5100 0    50   Output ~ 0
+EXTV
+Wire Wire Line
+	3450 5100 3150 5100
+Connection ~ 3450 5100
+Text HLabel 2000 6600 0    50   Output ~ 0
+COMVID
+Wire Wire Line
+	2000 6600 2200 6600
+$Comp
+L power:GND #PWR0138
+U 1 1 5DF966DD
+P 7550 1350
+F 0 "#PWR0138" H 7550 1100 50  0001 C CNN
+F 1 "GND" H 7555 1177 50  0000 C CNN
+F 2 "" H 7550 1350 50  0001 C CNN
+F 3 "" H 7550 1350 50  0001 C CNN
+	1    7550 1350
+	1    0    0    -1
+$EndComp
+Wire Wire Line
+	650  3650 2300 3650
+$Comp
+L Diode:1N4148 D1
+U 1 1 5E052EE5
+P 2650 3800
+F 0 "D1" H 2650 3584 50  0000 C CNN
+F 1 "1N4148" H 2650 3675 50  0000 C CNN
+F 2 "Diode_THT:D_DO-35_SOD27_P7.62mm_Horizontal" H 2650 3625 50  0001 C CNN
+F 3 "https://assets.nexperia.com/documents/data-sheet/1N4148_1N4448.pdf" H 2650 3800 50  0001 C CNN
+	1    2650 3800
+	-1   0    0    1
+$EndComp
+Wire Wire Line
+	2500 3800 2300 3800
+Wire Wire Line
+	2800 3800 3000 3800
+Connection ~ 7700 3000
 $Comp
 L Z80MiniFrame-Sound_Graphics-rescue:AS6C62256-55PCN-Memory_RAM U5
@@
 	1    0    0    -1
 $EndComp
-$Comp
-L 74xx:74LS574 U3
-U 1 1 5D7A0CA0
-P 6600 3600
-F 0 "U3" H 6600 4581 50  0000 C CNN
-F 1 "74LS574" H 6600 4490 50  0000 C CNN
-F 2 "Package_DIP:DIP-20_W7.62mm_Socket_LongPads" H 6600 3600 50  0001 C CNN
-F 3 "http://www.ti.com/lit/gpn/sn74LS574" H 6600 3600 50  0001 C CNN
-	1    6600 3600
-	1    0    0    -1
-$EndComp
-$Comp
-L Device:CTRIM CV1
-U 1 1 5DF8BFF1
-P 1350 2850
-F 0 "CV1" V 1603 2850 50  0000 C CNN
-F 1 "5-50pF" V 1512 2850 50  0000 C CNN
-F 2 "Potentiometer_THT:Potentiometer_ACP_CA9-V10_Vertical" H 1350 2850 50  0001 C CNN
-F 3 "~" H 1350 2850 50  0001 C CNN
-	1    1350 2850
-	0    -1   -1   0
-$EndComp
-Connection ~ 1750 2850
-$Comp
-L power:GND #PWR0129
-U 1 1 5E069747
-P 1750 3150
-F 0 "#PWR0129" H 1750 2900 50  0001 C CNN
-F 1 "GND" H 1755 2977 50  0000 C CNN
-F 2 "" H 1750 3150 50  0001 C CNN
-F 3 "" H 1750 3150 50  0001 C CNN
-	1    1750 3150
-	1    0    0    -1
-$EndComp
-Wire Wire Line
-	2450 2550 2450 3200
-Wire Wire Line
-	2450 3200 3000 3200
-Wire Wire Line
-	3000 3300 1950 3300
-Wire Wire Line
-	1950 3300 1950 2850
-Wire Wire Line
-	1950 2850 1750 2850
-Text HLabel 3150 5100 0    50   Output ~ 0
-EXTV
-Wire Wire Line
-	3450 5100 3150 5100
-Connection ~ 3450 5100
-Text HLabel 2000 6600 0    50   Output ~ 0
-COMVID
-Wire Wire Line
-	2000 6600 2200 6600
-$Comp
-L power:GND #PWR0138
-U 1 1 5DF966DD
-P 7550 1350
-F 0 "#PWR0138" H 7550 1100 50  0001 C CNN
-F 1 "GND" H 7555 1177 50  0000 C CNN
-F 2 "" H 7550 1350 50  0001 C CNN
-F 3 "" H 7550 1350 50  0001 C CNN
-	1    7550 1350
-	1    0    0    -1
-$EndComp
-Wire Wire Line
-	650  3650 2300 3650
-$Comp
-L Diode:1N4148 D1
-U 1 1 5E052EE5
-P 2650 3800
-F 0 "D1" H 2650 3584 50  0000 C CNN
-F 1 "1N4148" H 2650 3675 50  0000 C CNN
-F 2 "Diode_THT:D_DO-35_SOD27_P7.62mm_Horizontal" H 2650 3625 50  0001 C CNN
-F 3 "https://assets.nexperia.com/documents/data-sheet/1N4148_1N4448.pdf" H 2650 3800 50  0001 C CNN
-	1    2650 3800
-	-1   0    0    1
-$EndComp
-Wire Wire Line
-	2500 3800 2300 3800
-Wire Wire Line
-	2800 3800 3000 3800
+Wire Bus Line
+	7700 3000 9250 3000
+Wire Wire Line
+	3950 4100 4100 4100
+Wire Wire Line
+	4100 4100 4100 5800
+Wire Wire Line
+	4100 5800 3150 5800
+Wire Wire Line
+	3950 2350 4250 2350
 Wire Wire Line
 	9000 1450 9800 1450
 Wire Wire Line
 	9000 1950 9700 1950
-Wire Wire Line
-	3950 2350 4250 2350
 Wire Wire Line
 	7550 1350 8000 1350
@@
 Wire Bus Line
 	9250 1050 9250 1950
-Wire Bus Line
-	7800 1050 7800 2150
 Wire Bus Line
 	7700 3000 7700 6850
@@
 	4150 3350 4150 6850
 Wire Bus Line
+	7800 1050 7800 2150
+Wire Bus Line
 	7350 1050 7350 3700
 Wire Bus Line
 	5850 1050 5850 5550
+Text HLabel 3150 5800 0    50   Output ~ 0
+CPUCLK
 $EndSCHEMATC
