File: schematics/Z80Mini/serial_adapter/serialadapter/serialadapter.kicad_pcb (KiCad board)
At the start: 2 copper layers, 86.4 x 57.1 mm, 25 parts, among them J1 TTL Serial, J2 RS232, J3 USB_B, J4 I2C, U1 MAX3222CPN+, U2 74LS365, U3 MCP2221A-I_SL

Commit message: Latest code changes and modified Makefile to support burn to EPROM Emulator
Connections:
- U3 pad 5: /RX -> /TX
- U3 pad 6: /TX -> /RX
Routing:
- net /RX: track 74.1 -> 65.0 mm
- net VCC: track 200.4 -> 207.3 mm, vias 1 -> 2
- net /TX: track 78.8 -> 84.2 mm
Other:
- net class VCC added: clearance 0.2, trace_width 1, via_dia 0.8, via_drill 0.4
