File: schematics/Z80Mini/serial_adapter/serialadapter/serialadapter.sch (KiCad schematic (older format))
At the start: 23 parts, among them J1 TTL Serial, J2 RS232, J3 USB_B, J4 I2C, U1 MAX3222CPN+, U2 74LS365, U3 MCP2221A-I_SL

Commit message: Latest code changes and modified Makefile to support burn to EPROM Emulator
Connections:
- net RX: now also U3.6 (UTX); no longer U3.5 (URX)
- net TX: now also U3.5 (URX); no longer U3.6 (UTX)
Changed lines of the file:
@@
 Wire Wire Line
 	9750 4600 10150 4600
+Text Label 10150 4600 0    50   ~ 0
+RX
 Text Label 10150 4700 0    50   ~ 0
-RX
-Text Label 10150 4600 0    50   ~ 0
 TX
 Wire Wire Line

Commit message: Latest changes on reserved word tokens bugfixes
Parts:
- U1: symbol Interface_UART:MAX3222CPN+ -> serialadapter-rescue:MAX3222CPN+-Interface_UART
- U3: symbol Interface_USB:MCP2221A-I_SL -> serialadapter-rescue:MCP2221A-I_SL-Interface_USB
Changed lines of the file:
@@
 EESchema Schematic File Version 4
+LIBS:serialadapter-cache
 EELAYER 30 0
 EELAYER END
@@
 $EndComp
 $Comp
-L Interface_UART:MAX3222CPN+ U1
+L serialadapter-rescue:MAX3222CPN+-Interface_UART U1
 U 1 1 5F185A71
 P 5350 2450
@@
 $EndComp
 $Comp
-L Interface_USB:MCP2221A-I_SL U3
+L serialadapter-rescue:MCP2221A-I_SL-Interface_USB U3
 U 1 1 5F200371
 P 9150 4900
