File: schematics/Z80Allinone/Z80AllInOne/Z80AllInOne.kicad_pcb (KiCad board)
At the start: 4 copper layers, 393.7 x 209.6 mm, 169 parts, among them J1 USB_B_Micro, J10 CF Card IDE, J2 USER_IO_CONN, J3 COMP_VIDEOUT, J4 TTL SERIAL, J5 Conn_01x03_Male, J6 CASETTE/AUDIO, J7 KEYBOARD_HEADER, J8 Conn_01x07_Male, J9 9VDC, K1 ADW11, Q1 IRLML6402, Q2 2N3904, Q3 BC337, Q4 BC337, SW1 SW_DIP_x04, SW2 RESET, U1 Z80CPU, U10 74LS574, U11 AS6C62256-55PCN, U12 7400, U13 7400, U14 74LS138, U15 74LS139, U16 74LS32, U17 74HC04, U2 TC55257CPI, U20 74LS02, U21 AY-3-8910, U22 LM386, U23 NA555P, U24 Z80-CTC, U25 74LS32, U26 74LS148, U27 74HC00, U28 74LS373, U29 L7805, U3 28C256, U4 82C55A, U5 16550, U6 FT232RL, U7 TMS9918A, U8 74LS574, U9 74LS574, X1 4MHz, Y2 10.73MHz

Commit message: Latest all in one PCB improvements
Parts:
- moved D9 41.8 mm to (280.0, 34.9)
- moved C47 37.1 mm to (268.4, 48.3)
- moved D10 36.9 mm to (233.0, 73.0), turned to -90 degrees
- moved D7 36.1 mm to (298.4, 50.8)
- moved K1 36.1 mm to (293.4, 43.3)
- moved D8 35.2 mm to (280.0, 38.1)
- moved C34 33.5 mm to (346.7, 79.3)
- moved C35 33.5 mm to (317.5, 79.4)
- moved C36 33.5 mm to (318.8, 61.0)
- moved C46 33.5 mm to (309.9, 61.0)
- moved R16 33.5 mm to (342.9, 71.7)
- moved R20 33.5 mm to (337.8, 71.7)
- moved R21 33.5 mm to (327.7, 79.4)
- moved R22 33.5 mm to (332.7, 71.7)
- moved U12 33.5 mm to (302.3, 66.0)
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Routing:
- net GND: track 290.8 -> 199.8 mm, vias 6 -> 5
- net Net-(Q3-Pad1): track 35.7 -> 82.6 mm
- net Net-(C34-Pad1): track 75.1 -> 120.8 mm
- net Net-(U10-Pad1): track 249.2 -> 207.7 mm
- net /IO/Casette Interface/M1: track 115.8 -> 75.5 mm
- net /IO/Casette Interface/M2: track 104.8 -> 78.6 mm
- net /IO/PA6: track 164.6 -> 190.7 mm, vias 1 -> 2
- net /IO/Casette Interface/PC7: track 84.5 -> 110.2 mm
- net VCC: track 2034.5 -> 2059.4 mm, vias 7 -> 5
- net Net-(D7-Pad1): track 17.0 -> 41.3 mm
- net /IO/Casette Interface/PC6: track 95.1 -> 116.2 mm
- net /IO/Casette Interface/PC4: track 85.0 -> 104.4 mm, vias 0 -> 1
- net /IO/PA7: track 202.5 -> 185.3 mm
- net /IO/Casette Interface/PC3: track 77.7 -> 94.3 mm
- net /IO/Casette Interface/PC2: track 86.4 -> 102.8 mm, vias 0 -> 1
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Other:
- board text added: "Z80AIO4323210"

Commit message: Latest modifications of All-in-one PCB
Parts:
- removed D5: 1N4148, Diode_THT:D_DO-35_SOD27_P7.62mm_Horizontal
- removed J5: Conn_01x03_Male, Connector_PinHeader_2.54mm:PinHeader_1x03_P2.54mm_Vertical
- removed J9: 9VDC, TerminalBlock:TerminalBlock_bornier-2_P5.08mm
- removed JP4: PREAMP_MONO, Connector_PinHeader_2.54mm:PinHeader_2x03_P2.54mm_Vertical
- added C53: 100uF, Capacitor_THT:CP_Radial_D8.0mm_P3.80mm, F.Cu at (372.8, 75.6)
- added C54: 10uF, Capacitor_THT:CP_Radial_D8.0mm_P3.80mm, F.Cu at (383.0, 75.6)
- added D12: DIODE, Diode_THT:D_A-405_P7.62mm_Horizontal, F.Cu at (371.5, 38.7)
- C44: value 47uF -> 0.1uF
- C45: value 4.7uF -> 0.1uF
- J2: value USER_IO_CONN -> IDC_IO_CONN
- J8: value Conn_01x07_Male -> TRGS/TOS
- R42: footprint Resistor_THT:R_Axial_DIN0207_L6.3mm_D2.5mm_P7.62mm_Horizontal -> Resistor_THT:R_Axial_DIN0207_L6.3mm_D2.5mm_P10.16mm_Horizontal
- moved JP5 24.2 mm to (392.4, 55.2)
- moved C44 20.0 mm to (384.8, 61.0)
- moved D3 14.6 mm to (380.4, 67.9)
- moved C45 13.1 mm to (372.8, 86.4)
- moved R15 11.3 mm to (33.7, 72.4), turned to -90 degrees
- moved C33 10.4 mm to (29.8, 82.5), turned to 90 degrees
- moved C20 8.89 mm to (114.3, 132.1)
- moved C43 8.89 mm to (21.6, 78.7)
- moved SPEAKER1 7.62 mm to (24.1, 67.3)
- moved R14 7.24 mm to (41.3, 98.4)
- moved C23 7.13 mm to (132.1, 135.9), turned to 90 degrees
- moved C32 7.06 mm to (21.0, 109.2)
- moved R13 6.63 mm to (31.1, 101.6)
- moved U29 6.54 mm to (372.7, 57.9)
- moved C42 6.10 mm to (27.9, 108.9)
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Connections:
- JP5 pad 1: GND -> Net-(D3-Pad1)
- JP5 pad 2: Net-(J9-Pad2) -> GND
- JP5 pad 3: Net-(D3-Pad1) -> GND
- R12 pad 2: Net-(JP4-Pad1) -> Net-(R12-Pad2)
- R13 pad 2: Net-(JP4-Pad1) -> Net-(R12-Pad2)
- U21 pad 3: Net-(J5-Pad2) -> Net-(R12-Pad2)
- U21 pad 38: Net-(J5-Pad1) -> Net-(R12-Pad2)
- U21 pad 4: Net-(J5-Pad3) -> Net-(R12-Pad2)
- U7 pad 16: Net-(D5-Pad1) -> /VDP_INT
Routing:
- net GND: track 199.8 -> 155.1 mm, vias 5 -> 6
- net Net-(R12-Pad2): track 0.00 -> 41.7 mm
- net /VIDEO/VD0: track 66.5 -> 105.8 mm, vias 0 -> 2
- net Net-(J5-Pad1): track 35.7 -> 0.00 mm
- net /VIDEO/VD1: track 66.4 -> 99.6 mm, vias 0 -> 2
- net /VDP_INT: track 150.2 -> 182.5 mm
- net /VIDEO/VD2: track 66.5 -> 93.2 mm, vias 0 -> 2
- net Net-(J5-Pad2): track 22.5 -> 0.00 mm
- net /BUS Expansion/D3: track 810.4 -> 832.3 mm
- net Net-(J5-Pad3): track 21.5 -> 0.00 mm
- net Net-(D5-Pad1): track 20.9 -> 0.00 mm
- net Net-(J9-Pad2): track 20.3 -> 0.00 mm
- net Net-(JP4-Pad1): track 19.6 -> 0.00 mm
- net /VIDEO/VD3: track 81.1 -> 100.0 mm, vias 0 -> 1
- net /VIDEO/AD3: track 88.4 -> 106.7 mm
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Other:
- copper layers 4 -> 2

Commit message: Latest changes for adapt source to support Z80AllInOne adding some macros and latest schematic improvements
Parts:
- added ?: , , F.Cu at (214.6, 146.1)
- added ?: , , F.Cu at (396.2, 39.4)
- added ?: , , F.Cu at (399.4, 153.7)
- added J5: USR_INTR, Connector_PinHeader_2.54mm:PinHeader_1x04_P2.54mm_Vertical, F.Cu at (215.9, 179.1)
- added JP4: MREQ/A8, Connector_PinHeader_2.54mm:PinHeader_1x03_P2.54mm_Vertical, F.Cu at (248.9, 194.9)
- added JP6: INTRA, Connector_PinHeader_2.54mm:PinHeader_1x03_P2.54mm_Vertical, F.Cu at (227.3, 83.2)
- J2: value IDC_IO_CONN -> USER_IO_CONN
- JP1: value USB_POWER -> USB_POWER_SW
- K1: value ADW11 -> FINDER-30.22; footprint Relay_THT:Relay_1P1T_NO_10x24x18.8mm_Panasonic_ADW11xxxxW_THT -> Relay_THT:Relay_DPDT_Finder_30.22
- R11: footprint Resistor_THT:R_Axial_DIN0207_L6.3mm_D2.5mm_P7.62mm_Horizontal -> Resistor_THT:R_Axial_DIN0207_L6.3mm_D2.5mm_P10.16mm_Horizontal
- R4, R5, R6, R7: value R -> 1K2
- RN1: value R_Network08 -> 4K7
- U2: value TC55257CPI -> MAIN RAM
- U29: footprint Package_TO_SOT_THT:TO-126-3_Horizontal_TabDown -> Package_TO_SOT_THT:TO-220-3_Horizontal_TabDown
- moved R44 71.4 mm to (336.6, 189.6), turned to 0 degrees
- moved C19 58.2 mm to (179.2, 48.3)
- moved R1 43.2 mm to (330.2, 106.7)
- moved R2 43.2 mm to (320.0, 106.7)
- moved R3 43.2 mm to (325.1, 106.7)
- moved C10 35.8 mm to (381.0, 123.2)
- moved C7 35.8 mm to (369.6, 147.3)
- moved C8 35.8 mm to (364.5, 144.8)
- moved C9 35.8 mm to (377.2, 128.3)
- moved FB1 35.8 mm to (377.4, 144.8)
- moved JP2 35.8 mm to (367.0, 152.4)
- moved Q1 35.8 mm to (370.8, 143.5)
- moved R10 35.8 mm to (364.2, 136.0)
- moved U6 35.8 mm to (368.0, 125.8)
- moved JP1 35.7 mm to (392.4, 152.4)
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Connections:
- net /INT_DEV2 renamed /PPI_INT
- U13 pad 3: Net-(U13-Pad3) -> Net-(JP4-Pad3)
- U14 pad 6: Net-(U13-Pad3) -> Net-(JP4-Pad2)
- U15 pad 2: GND -> /IO/A15
- U15 pad 3: /IO/A15 -> GND
- U18 pad 11: /IO/Casette Interface/PC3 -> Net-(U18-Pad11)
- U2 pad 20: /ROM_CE -> /RAM_CE
- U3 pad 20: /RAM_CE -> /ROM_CE
Routing:
- net VCC: track 2047.1 -> 1919.4 mm, vias 5 -> 8
- net /IO/A0: track 851.9 -> 744.3 mm
- net /IO/A1: track 785.4 -> 692.3 mm
- net /PPI_INT: track 23.7 -> 115.7 mm
- net /NMI: track 553.4 -> 634.2 mm, vias 2 -> 4
- net Net-(C19-Pad1): track 74.2 -> 5.58 mm
- net /PPI_CE: track 343.5 -> 275.7 mm
- net /IORQ: track 541.0 -> 480.3 mm, vias 6 -> 5
- net Net-(C19-Pad2): track 11.3 -> 69.3 mm
- net /IO/A8: track 472.3 -> 419.0 mm
- net /BUSACK: track 571.6 -> 520.5 mm
- net /BUS Expansion/D0: track 782.4 -> 731.9 mm
- net /HALT: track 531.5 -> 481.7 mm
- net /M1: track 526.6 -> 476.8 mm
- net /BUS Expansion/D1: track 793.1 -> 744.2 mm
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Other:
- board size 393.7 x 209.6 mm -> 389.9 x 174 mm
- board text added: "Device Map: 0x0000 PPI 0x0020 UART 0x0040 VDP 0x0060 PSG 0x0080 CTC 0x00A0 CF 0x00C0 External"
- board text added: "TOMEU CAPÓ 2022 (C) BOTILLA TECHs"
- board text added: "Z80 MiniFrame All-in-one v1.0.1 (TCC 2022)"
- board text removed: "Device Map: 0x0000 PPI 0x0010 UART 0x0020 VDP 0x0030 PSG 0x0040 CTC 0x0050 CF 0x0060 External"
- board text removed: "Z80 MiniFrame All-in-one v1.0 (TCC 2022)"
