File: schematics/Z80Allinone/Z80AllInOne/reset.kicad_sch (KiCad schematic)
At the start: 14 parts, among them Q3 BC337, SW2 RESET, U12 7400, U23 NA555P

Commit message: Latest changes and replace CTC for 8253 PIT
Parts:
- removed U23: NA555P, Package_DIP:DIP-8_W7.62mm, symbol Timer:NA555P
- added U23: NE556, Package_DIP:DIP-14_W7.62mm_LongPads, symbol Timer:NE556
Connections:
- net GND: now also U23.7 (GND)
- net VCC: now also U23.10 (R), U23.14 (VCC)
- net at C34.1, R16.2, SW2.2: now also U23.8 (TR)
- net at U12.1, U12.2: now also U23.9 (Q)
- net at C36.1, R20.2: now also U23.12 (THR), U23.13 (DIS)
Changed lines of the file:
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@@
     (pin "2")
+  )
+  (symbol (lib_id "Timer:NE556") (at 132.08 90.17 0) (unit 2)
+    (in_bom yes) (on_board yes) (fields_autoplaced)
+    (property "Reference" "U23" (id 0) (at 134.0994 77.47 0)
+      (effects (font (size 1.27 1.27)) (justify left))
+    )
+    (property "Value" "NE556" (id 1) (at 134.0994 80.01 0)
+      (effects (font (size 1.27 1.27)) (justify left))
+    )
+    (property "Footprint" "Package_DIP:DIP-14_W7.62mm_LongPads" (id 2) (at 132.08 90.17 0)
+      (effects (font (size 1.27 1.27)) hide)
+    )
+    (property "Datasheet" "http://www.ti.com/lit/ds/symlink/ne556.pdf" (id 3) (at 132.08 90.17 0)
+      (effects (font (size 1.27 1.27)) hide)
+    )
+    (pin "14")
+    (pin "7")
+    (pin "1")
+    (pin "2")
+    (pin "3")
+    (pin "4")
+    (pin "5")
+    (pin "6")
+    (pin "10")
+    (pin "11")
+    (pin "12")
+    (pin "13")
+    (pin "8")
+    (pin "9")
   )
   (symbol (lib_id "power:VCC") (at 148.59 72.39 0) (unit 1)
@@
     (pin "1")
   )
-  (symbol (lib_id "Timer:NA555P") (at 132.08 90.17 0) (unit 1)
-    (in_bom yes) (on_board yes) (fields_autoplaced)
-    (property "Reference" "U23" (id 0) (at 134.0994 77.47 0)
-      (effects (font (size 1.27 1.27)) (justify left))
-    )
-    (property "Value" "NA555P" (id 1) (at 134.0994 80.01 0)
-      (effects (font (size 1.27 1.27)) (justify left))
-    )
-    (property "Footprint" "Package_DIP:DIP-8_W7.62mm" (id 2) (at 148.59 100.33 0)
-      (effects (font (size 1.27 1.27)) hide)
-    )
-    (property "Datasheet" "http://www.ti.com/lit/ds/symlink/ne555.pdf" (id 3) (at 153.67 100.33 0)
-      (effects (font (size 1.27 1.27)) hide)
-    )
-    (pin "1")
-    (pin "8")
-    (pin "2")
-    (pin "3")
-    (pin "4")
-    (pin "5")
-    (pin "6")
-    (pin "7")
-  )
   (symbol (lib_id "74xx:7400") (at 193.04 85.09 0) (unit 2)
